File: _autosave-DaisySeedBreakout.kicad_pcb (KiCad board)
At the start: 2 copper layers, 56.8 x 65 mm, 126 parts, among them J1 Conn_01x03, J10 Conn_01x03, J15 Conn_01x03, J17 Pins_02x10_P2.54mm_TH, J19 Pins_02x10_P2.54mm_TH, J2 Conn_01x02, J23 Pins_02x10_P2.54mm_TH, J26 Pins_02x10_P2.54mm_TH, J27 Pins_02x10_P2.54mm_TH, J28 Pins_02x10_P2.54mm_TH, J29 Pins_02x10_P2.54mm_TH, J3 Conn_01x03, J35 Conn_01x02, J4 5027740891, J6 Conn_01x02, J7 Pins_02x10_P2.54mm_TH, J8 Conn_01x02, J9 Conn_01x02, U1 H11L1M, U10 TPD2EUSB30ADRTR, U2 PAM8320RDR, U4 ATMEGA1608-MFR, U5 MAX9814, U6 DSC6001CE2A-010.0000, U7 TLV9062IDR

Commit message: commit before simplifyting the board further
Parts:
- added A1: Electrosmith_Daisy_Seed_Rev4, Module:Electrosmith_Daisy_Seed, F.Cu at (517.9, 60.5)
- added A1: Electrosmith_Daisy_Seed_Rev4, Module:Electrosmith_Daisy_Seed, F.Cu at (190.6, 45.9)
- added A1: Electrosmith_Daisy_Seed_Rev4, Module:Electrosmith_Daisy_Seed, F.Cu at (245.4, 44.7)
- added C12: 10U, Capacitor_SMD:C_0805_2012Metric, F.Cu at (497.1, 67.2)
- added C12: 10U, Capacitor_SMD:C_0805_2012Metric, F.Cu at (252.1, 65.5)
- added C12: 10U, Capacitor_SMD:C_0805_2012Metric, F.Cu at (197.2, 66.8)
- added C13: 10U, Capacitor_SMD:C_0805_2012Metric, F.Cu at (506.1, 67.6)
- added C13: 10U, Capacitor_SMD:C_0805_2012Metric, F.Cu at (197.6, 57.8)
- added C13: 10U, Capacitor_SMD:C_0805_2012Metric, F.Cu at (252.5, 56.5)
- added C14: 0.1uF, Capacitor_SMD:C_0402_1005Metric, F.Cu at (195.3, 71.5)
- added C14: 0.1uF, Capacitor_SMD:C_0402_1005Metric, F.Cu at (250.2, 70.3)
- added C14: 0.1uF, Capacitor_SMD:C_0402_1005Metric, F.Cu at (492.3, 65.3)
- added C15: 10U, Capacitor_SMD:C_0805_2012Metric, F.Cu at (503.9, 67.7)
- added C15: 10U, Capacitor_SMD:C_0805_2012Metric, F.Cu at (252.6, 58.7)
- added C15: 10U, Capacitor_SMD:C_0805_2012Metric, F.Cu at (197.7, 59.9)
- added C16: 10U, Capacitor_SMD:C_0805_2012Metric, F.Cu at (199.4, 66.8)
- added C16: 10U, Capacitor_SMD:C_0805_2012Metric, F.Cu at (497.0, 69.4)
- added C16: 10U, Capacitor_SMD:C_0805_2012Metric, F.Cu at (254.2, 65.6)
- added C3: 0.1uF, Capacitor_SMD:C_0402_1005Metric, F.Cu at (201.4, 47.7)
- added C3: 0.1uF, Capacitor_SMD:C_0402_1005Metric, F.Cu at (256.2, 46.4)
- added C3: 0.1uF, Capacitor_SMD:C_0402_1005Metric, F.Cu at (516.2, 71.3)
- added C32: 860020474014, 470uF:CAP_WCAP-ATG5_8x11.5_WRE, F.Cu at (358.1, 94.0)
- added C32: 860020474014, 470uF:CAP_WCAP-ATG5_8x11.5_WRE, F.Cu at (213.9, 62.8)
- added C6: 0.1uF, Capacitor_SMD:C_0603_1608Metric, F.Cu at (518.2, 70.6)
- added C6: 0.1uF, Capacitor_SMD:C_0603_1608Metric, F.Cu at (255.5, 44.5)
- added C6: 0.1uF, Capacitor_SMD:C_0603_1608Metric, F.Cu at (200.6, 45.7)
- added H1: MountingHole, MountingHole:MountingHole_3.2mm_M3_DIN965_Pad, F.Cu at (516.1, 38.6)
- added H1: MountingHole, MountingHole:MountingHole_3.2mm_M3_DIN965_Pad, F.Cu at (228.8, 45.9)
- added H1: MountingHole, MountingHole:MountingHole_3.2mm_M3_DIN965_Pad, F.Cu at (174.0, 47.2)
- added H2: MountingHole, MountingHole:MountingHole_3.2mm_M3_DIN965_Pad, F.Cu at (213.0, 92.6)
- added H2: MountingHole, MountingHole:MountingHole_3.2mm_M3_DIN965_Pad, F.Cu at (267.1, 91.2)
- added H2: MountingHole, MountingHole:MountingHole_3.2mm_M3_DIN965_Pad, F.Cu at (459.1, 82.5)
- added H3: MountingHole, MountingHole:MountingHole_3.2mm_M3_DIN965_Pad, F.Cu at (173.3, 92.3)
- added H3: MountingHole, MountingHole:MountingHole_3.2mm_M3_DIN965_Pad, F.Cu at (459.6, 38.9)
- added H3: MountingHole, MountingHole:MountingHole_3.2mm_M3_DIN965_Pad, F.Cu at (228.2, 91.1)
- added H4: MountingHole, MountingHole:MountingHole_3.2mm_M3_DIN965_Pad, F.Cu at (215.0, 47.6)
- added H4: MountingHole, MountingHole:MountingHole_3.2mm_M3_DIN965_Pad, F.Cu at (516.0, 82.5)
- added H4: MountingHole, MountingHole:MountingHole_3.2mm_M3_DIN965_Pad, F.Cu at (267.3, 46.4)
- added J1: Conn_01x03, Ultralibrarian:PinHeader_1x03_P2.54mm_Vertical_Female, F.Cu at (463.6, 54.8)
- added J1: Conn_01x03, Ultralibrarian:PinHeader_1x03_P2.54mm_Vertical_Female, F.Cu at (240.3, 69.7)
- added J1: Conn_01x03, Ultralibrarian:PinHeader_1x03_P2.54mm_Vertical_Female, F.Cu at (463.6, 59.9)
- added J1: Conn_01x03, Ultralibrarian:PinHeader_1x03_P2.54mm_Vertical_Female, F.Cu at (231.5, 74.8)
- added J1: Conn_01x03, Ultralibrarian:PinHeader_1x03_P2.54mm_Vertical_Female, F.Cu at (240.3, 64.6)
- added J1: Conn_01x03, Ultralibrarian:PinHeader_1x03_P2.54mm_Vertical_Female, F.Cu at (463.6, 64.9)
- added J1: Conn_01x03, Ultralibrarian:PinHeader_1x03_P2.54mm_Vertical_Female, F.Cu at (185.4, 71.0)
- added J1: Conn_01x03, Ultralibrarian:PinHeader_1x03_P2.54mm_Vertical_Female, F.Cu at (494.7, 84.4)
- added J1: Conn_01x03, Ultralibrarian:PinHeader_1x03_P2.54mm_Vertical_Female, F.Cu at (185.4, 55.7)
- added J1: Conn_01x03, Ultralibrarian:PinHeader_1x03_P2.54mm_Vertical_Female, F.Cu at (463.6, 70.0)
- added J1: Conn_01x03, Ultralibrarian:PinHeader_1x03_P2.54mm_Vertical_Female, F.Cu at (185.4, 50.6)
- added J1: Conn_01x03, Ultralibrarian:PinHeader_1x03_P2.54mm_Vertical_Female, F.Cu at (240.3, 49.4)
- added J1: Conn_01x03, Ultralibrarian:PinHeader_1x03_P2.54mm_Vertical_Female, F.Cu at (185.4, 65.9)
- added J1: Conn_01x03, Ultralibrarian:PinHeader_1x03_P2.54mm_Vertical_Female, F.Cu at (184.8, 85.2)
- added J1: Conn_01x03, Ultralibrarian:PinHeader_1x03_P2.54mm_Vertical_Female, F.Cu at (463.6, 49.7)
- added J1: Conn_01x03, Ultralibrarian:PinHeader_1x03_P2.54mm_Vertical_Female, F.Cu at (185.4, 60.8)
- added J1: Conn_01x03, Ultralibrarian:PinHeader_1x03_P2.54mm_Vertical_Female, F.Cu at (240.3, 59.5)
- added J1: Conn_01x03, Ultralibrarian:PinHeader_1x03_P2.54mm_Vertical_Female, F.Cu at (240.3, 54.5)
- added J10: Conn_01x03, Ultralibrarian:PinHeader_1x03_P2.54mm_Vertical_Female, F.Cu at (339.2, 107.7)
- added J15: Conn_01x03, Ultralibrarian:PinHeader_1x03_P2.54mm_Vertical_Female, F.Cu at (211.2, 54.5)
- added J15: Conn_01x03, Ultralibrarian:PinHeader_1x03_P2.54mm_Vertical_Female, F.Cu at (510.6, 84.4)
- added J15: Conn_01x03, Ultralibrarian:PinHeader_1x03_P2.54mm_Vertical_Female, F.Cu at (266.7, 58.4)
- added J18: ~, Ultralibrarian:STX-4235-3-3-N, F.Cu at (304.9, 17.9)
- added J18: ~, Ultralibrarian:STX-4235-3-3-N, F.Cu at (517.5, 49.5)
- added J2: Conn_01x02, 1x2FemaleVertical:PinHeader_1x02_P2.54mm_VerticalFemale, F.Cu at (268.9, 75.4)
- added J2: Conn_01x02, 1x2FemaleVertical:PinHeader_1x02_P2.54mm_VerticalFemale, F.Cu at (268.9, 78.0)
- added J2: Conn_01x02, 1x2FemaleVertical:PinHeader_1x02_P2.54mm_VerticalFemale, F.Cu at (175.1, 86.2)
- added J2: Conn_01x02, 1x2FemaleVertical:PinHeader_1x02_P2.54mm_VerticalFemale, F.Cu at (175.3, 76.2)
- added J2: Conn_01x02, 1x2FemaleVertical:PinHeader_1x02_P2.54mm_VerticalFemale, F.Cu at (175.3, 78.7)
- added J2: Conn_01x02, 1x2FemaleVertical:PinHeader_1x02_P2.54mm_VerticalFemale, F.Cu at (182.5, 76.2)
- added J2: Conn_01x02, 1x2FemaleVertical:PinHeader_1x02_P2.54mm_VerticalFemale, F.Cu at (502.2, 55.4)
- added J2: Conn_01x02, 1x2FemaleVertical:PinHeader_1x02_P2.54mm_VerticalFemale, F.Cu at (504.7, 55.4)
- added J2: Conn_01x02, 1x2FemaleVertical:PinHeader_1x02_P2.54mm_VerticalFemale, F.Cu at (175.2, 83.6)
- added J2: Conn_01x02, 1x2FemaleVertical:PinHeader_1x02_P2.54mm_VerticalFemale, F.Cu at (502.1, 45.2)
- added J2: Conn_01x02, 1x2FemaleVertical:PinHeader_1x02_P2.54mm_VerticalFemale, F.Cu at (269.0, 83.3)
- added J2: Conn_01x02, 1x2FemaleVertical:PinHeader_1x02_P2.54mm_VerticalFemale, F.Cu at (504.6, 45.2)
- added J2: Conn_01x02, 1x2FemaleVertical:PinHeader_1x02_P2.54mm_VerticalFemale, F.Cu at (239.8, 83.4)
- added J2: Conn_01x02, 1x2FemaleVertical:PinHeader_1x02_P2.54mm_VerticalFemale, F.Cu at (268.9, 85.8)
- added J2: Conn_01x02, 1x2FemaleVertical:PinHeader_1x02_P2.54mm_VerticalFemale, F.Cu at (510.5, 40.2)
- added J2: Conn_01x02, 1x2FemaleVertical:PinHeader_1x02_P2.54mm_VerticalFemale, F.Cu at (239.8, 80.8)
- added J3: Conn_01x03, Ultralibrarian:PinHeader_1x03_P2.54mm_Vertical_Female, F.Cu at (185.4, 68.4)
- added J3: Conn_01x03, Ultralibrarian:PinHeader_1x03_P2.54mm_Vertical_Female, F.Cu at (185.4, 63.3)
- added J3: Conn_01x03, Ultralibrarian:PinHeader_1x03_P2.54mm_Vertical_Female, F.Cu at (268.7, 68.6)
- added J3: Conn_01x03, Ultralibrarian:PinHeader_1x03_P2.54mm_Vertical_Female, F.Cu at (240.3, 67.2)
- added J3: Conn_01x03, Ultralibrarian:PinHeader_1x03_P2.54mm_Vertical_Female, F.Cu at (463.6, 67.5)
- added J3: Conn_01x03, Ultralibrarian:PinHeader_1x03_P2.54mm_Vertical_Female, F.Cu at (469.9, 20.3)
- added J3: Conn_01x03, Ultralibrarian:PinHeader_1x03_P2.54mm_Vertical_Female, F.Cu at (185.4, 58.3)
- added J3: Conn_01x03, Ultralibrarian:PinHeader_1x03_P2.54mm_Vertical_Female, F.Cu at (185.4, 53.2)
- added J3: Conn_01x03, Ultralibrarian:PinHeader_1x03_P2.54mm_Vertical_Female, F.Cu at (463.6, 52.2)
- added J3: Conn_01x03, Ultralibrarian:PinHeader_1x03_P2.54mm_Vertical_Female, F.Cu at (467.4, 20.3)
- added J3: Conn_01x03, Ultralibrarian:PinHeader_1x03_P2.54mm_Vertical_Female, F.Cu at (240.3, 46.8)
- added J3: Conn_01x03, Ultralibrarian:PinHeader_1x03_P2.54mm_Vertical_Female, F.Cu at (463.6, 62.4)
- added J3: Conn_01x03, Ultralibrarian:PinHeader_1x03_P2.54mm_Vertical_Female, F.Cu at (463.6, 57.3)
- added J3: Conn_01x03, Ultralibrarian:PinHeader_1x03_P2.54mm_Vertical_Female, F.Cu at (184.8, 82.7)
- added J3: Conn_01x03, Ultralibrarian:PinHeader_1x03_P2.54mm_Vertical_Female, F.Cu at (240.3, 57.0)
- added J3: Conn_01x03, Ultralibrarian:PinHeader_1x03_P2.54mm_Vertical_Female, F.Cu at (494.7, 81.9)
- added J3: Conn_01x03, Ultralibrarian:PinHeader_1x03_P2.54mm_Vertical_Female, F.Cu at (482.6, 47.2)
- added J3: Conn_01x03, Ultralibrarian:PinHeader_1x03_P2.54mm_Vertical_Female, F.Cu at (240.3, 62.1)
- added J3: Conn_01x03, Ultralibrarian:PinHeader_1x03_P2.54mm_Vertical_Female, F.Cu at (240.4, 74.7)
- added J3: Conn_01x03, Ultralibrarian:PinHeader_1x03_P2.54mm_Vertical_Female, F.Cu at (185.4, 48.1)
- added J3: Conn_01x03, Ultralibrarian:PinHeader_1x03_P2.54mm_Vertical_Female, F.Cu at (482.6, 49.7)
- added J3: Conn_01x03, Ultralibrarian:PinHeader_1x03_P2.54mm_Vertical_Female, F.Cu at (216.0, 85.4)
- added J3: Conn_01x03, Ultralibrarian:PinHeader_1x03_P2.54mm_Vertical_Female, F.Cu at (463.6, 47.2)
- added J3: Conn_01x03, Ultralibrarian:PinHeader_1x03_P2.54mm_Vertical_Female, F.Cu at (216.0, 88.0)
- added J3: Conn_01x03, Ultralibrarian:PinHeader_1x03_P2.54mm_Vertical_Female, F.Cu at (266.1, 68.6)
- added J3: Conn_01x03, Ultralibrarian:PinHeader_1x03_P2.54mm_Vertical_Female, F.Cu at (240.3, 51.9)
- added J35: Conn_01x02, 1x2FemaleVertical:PinHeader_1x02_P2.54mm_VerticalFemale, F.Cu at (471.2, 54.8)
- added J35: Conn_01x02, 1x2FemaleVertical:PinHeader_1x02_P2.54mm_VerticalFemale, F.Cu at (230.1, 69.9)
- added J35: Conn_01x02, 1x2FemaleVertical:PinHeader_1x02_P2.54mm_VerticalFemale, F.Cu at (230.1, 59.7)
- added J35: Conn_01x02, 1x2FemaleVertical:PinHeader_1x02_P2.54mm_VerticalFemale, F.Cu at (478.8, 52.2)
- added J35: Conn_01x02, 1x2FemaleVertical:PinHeader_1x02_P2.54mm_VerticalFemale, F.Cu at (230.1, 54.6)
- added J35: Conn_01x02, 1x2FemaleVertical:PinHeader_1x02_P2.54mm_VerticalFemale, F.Cu at (175.3, 66.0)
- added J35: Conn_01x02, 1x2FemaleVertical:PinHeader_1x02_P2.54mm_VerticalFemale, F.Cu at (471.2, 49.7)
- added J35: Conn_01x02, 1x2FemaleVertical:PinHeader_1x02_P2.54mm_VerticalFemale, F.Cu at (175.3, 55.9)
- added J35: Conn_01x02, 1x2FemaleVertical:PinHeader_1x02_P2.54mm_VerticalFemale, F.Cu at (175.3, 61.0)
- added J35: Conn_01x02, 1x2FemaleVertical:PinHeader_1x02_P2.54mm_VerticalFemale, F.Cu at (175.3, 71.1)
- added J35: Conn_01x02, 1x2FemaleVertical:PinHeader_1x02_P2.54mm_VerticalFemale, F.Cu at (485.8, 84.4)
- added J35: Conn_01x02, 1x2FemaleVertical:PinHeader_1x02_P2.54mm_VerticalFemale, F.Cu at (230.1, 64.8)
- added J5: ~, Ultralibrarian:BladeFuseHolder, F.Cu at (472.7, 83.2)
- added J6: Conn_01x02, 1x2FemaleVertical:PinHeader_1x02_P2.54mm_VerticalFemale, F.Cu at (478.8, 49.7)
- added J6: Conn_01x02, 1x2FemaleVertical:PinHeader_1x02_P2.54mm_VerticalFemale, F.Cu at (230.1, 62.2)
- added J6: Conn_01x02, 1x2FemaleVertical:PinHeader_1x02_P2.54mm_VerticalFemale, F.Cu at (471.2, 52.2)
- added J6: Conn_01x02, 1x2FemaleVertical:PinHeader_1x02_P2.54mm_VerticalFemale, F.Cu at (214.9, 79.6)
- added J6: Conn_01x02, 1x2FemaleVertical:PinHeader_1x02_P2.54mm_VerticalFemale, F.Cu at (175.3, 63.5)
- added J6: Conn_01x02, 1x2FemaleVertical:PinHeader_1x02_P2.54mm_VerticalFemale, F.Cu at (230.1, 57.2)
- added J6: Conn_01x02, 1x2FemaleVertical:PinHeader_1x02_P2.54mm_VerticalFemale, F.Cu at (471.2, 47.2)
- added J6: Conn_01x02, 1x2FemaleVertical:PinHeader_1x02_P2.54mm_VerticalFemale, F.Cu at (478.8, 47.2)
- added J6: Conn_01x02, 1x2FemaleVertical:PinHeader_1x02_P2.54mm_VerticalFemale, F.Cu at (175.3, 53.3)
- added J6: Conn_01x02, 1x2FemaleVertical:PinHeader_1x02_P2.54mm_VerticalFemale, F.Cu at (478.8, 54.8)
- added J6: Conn_01x02, 1x2FemaleVertical:PinHeader_1x02_P2.54mm_VerticalFemale, F.Cu at (175.3, 58.4)
- added J6: Conn_01x02, 1x2FemaleVertical:PinHeader_1x02_P2.54mm_VerticalFemale, F.Cu at (230.1, 52.1)
- added J6: Conn_01x02, 1x2FemaleVertical:PinHeader_1x02_P2.54mm_VerticalFemale, F.Cu at (485.8, 81.9)
- added J6: Conn_01x02, 1x2FemaleVertical:PinHeader_1x02_P2.54mm_VerticalFemale, F.Cu at (175.3, 68.6)
- added J6: Conn_01x02, 1x2FemaleVertical:PinHeader_1x02_P2.54mm_VerticalFemale, F.Cu at (230.1, 67.3)
- added MK2: Microphone_Condenser, microphone:MIC_AOM-6545_PUI, F.Cu at (214.2, 71.4)
- added MK2: Microphone_Condenser, microphone:MIC_AOM-6545_PUI, F.Cu at (229.3, 81.7)
- added R21: 2M, Resistor_SMD:R_0402_1005Metric, F.Cu at (250.2, 58.9)
- added R21: 2M, Resistor_SMD:R_0402_1005Metric, F.Cu at (503.7, 65.3)
- added R21: 2M, Resistor_SMD:R_0402_1005Metric, F.Cu at (195.3, 60.2)
- added R22: 2M, Resistor_SMD:R_0402_1005Metric, F.Cu at (254.9, 70.4)
- added R22: 2M, Resistor_SMD:R_0402_1005Metric, F.Cu at (200.0, 71.6)
- added R22: 2M, Resistor_SMD:R_0402_1005Metric, F.Cu at (492.3, 70.0)
- added R23: 2M, Resistor_SMD:R_0402_1005Metric, F.Cu at (201.2, 81.2)
- added R23: 2M, Resistor_SMD:R_0402_1005Metric, F.Cu at (482.7, 71.1)
- added R23: 2M, Resistor_SMD:R_0402_1005Metric, F.Cu at (256.0, 80.0)
- added R30: 2M, Resistor_SMD:R_0402_1005Metric, F.Cu at (494.7, 67.3)
- added R30: 2M, Resistor_SMD:R_0402_1005Metric, F.Cu at (197.3, 69.1)
- added R30: 2M, Resistor_SMD:R_0402_1005Metric, F.Cu at (252.2, 67.9)
- added R31: 2M, Resistor_SMD:R_0402_1005Metric, F.Cu at (201.5, 79.3)
- added R31: 2M, Resistor_SMD:R_0402_1005Metric, F.Cu at (484.5, 71.4)
- added R31: 2M, Resistor_SMD:R_0402_1005Metric, F.Cu at (256.3, 78.1)
- added R32: 4.7k, Resistor_SMD:R_0402_1005Metric, F.Cu at (494.7, 65.6)
- added R32: 4.7k, Resistor_SMD:R_0402_1005Metric, F.Cu at (250.5, 67.9)
- added R32: 4.7k, Resistor_SMD:R_0402_1005Metric, F.Cu at (195.6, 69.2)
- added R33: 4.7k, Resistor_SMD:R_0402_1005Metric, F.Cu at (482.1, 65.0)
- added R33: 4.7k, Resistor_SMD:R_0402_1005Metric, F.Cu at (249.9, 80.5)
- added R33: 4.7k, Resistor_SMD:R_0402_1005Metric, F.Cu at (195.0, 81.7)
- added R48: 10k, Resistor_SMD:R_0402_1005Metric, F.Cu at (246.1, 72.5)
- added R49: 10k, Resistor_SMD:R_0402_1005Metric, F.Cu at (246.1, 74.4)
- added R5: 2M, Resistor_SMD:R_0402_1005Metric, F.Cu at (252.8, 63.2)
- added R5: 2M, Resistor_SMD:R_0402_1005Metric, F.Cu at (197.9, 64.4)
- added R5: 2M, Resistor_SMD:R_0402_1005Metric, F.Cu at (499.5, 67.9)
- added R50: 10k, Resistor_SMD:R_0402_1005Metric, F.Cu at (246.1, 76.4)
- added R51: 10k, Resistor_SMD:R_0402_1005Metric, F.Cu at (246.1, 78.4)
- added R52: 10, Resistor_SMD:R_0402_1005Metric, F.Cu at (321.0, 50.1)
- added R56: 0, Resistor_SMD:R_0402_1005Metric, F.Cu at (482.9, 67.0)
- added R56: 0, Resistor_SMD:R_0402_1005Metric, F.Cu at (251.9, 79.7)
- added R56: 0, Resistor_SMD:R_0402_1005Metric, F.Cu at (197.0, 81.0)
- added R59: 0, Resistor_SMD:R_0402_1005Metric, F.Cu at (492.3, 67.8)
- added R59: 0, Resistor_SMD:R_0402_1005Metric, F.Cu at (197.9, 71.6)
- added R59: 0, Resistor_SMD:R_0402_1005Metric, F.Cu at (252.7, 70.3)
- added R60: DNP, Resistor_SMD:R_0402_1005Metric, F.Cu at (256.7, 72.0)
- added R60: DNP, Resistor_SMD:R_0402_1005Metric, F.Cu at (201.8, 73.3)
- added R60: DNP, Resistor_SMD:R_0402_1005Metric, F.Cu at (490.6, 71.8)
- added R61: DNP, Resistor_SMD:R_0402_1005Metric, F.Cu at (199.1, 81.0)
- added R61: DNP, Resistor_SMD:R_0402_1005Metric, F.Cu at (253.9, 79.8)
- added R61: DNP, Resistor_SMD:R_0402_1005Metric, F.Cu at (482.9, 69.0)
- added U1: H11L1M, digikey-footprints:DIP-6_W7.62mm, F.Cu at (233.2, 87.6)
- added U1: H11L1M, digikey-footprints:DIP-6_W7.62mm, F.Cu at (178.3, 88.9)
- added U1: H11L1M, digikey-footprints:DIP-6_W7.62mm, F.Cu at (448.5, 88.2)
- added U7: TLV9062IDR, TLV9062:D0008A_N, F.Cu at (487.6, 68.4)
- added U7: TLV9062IDR, TLV9062:D0008A_N, F.Cu at (253.3, 75.0)
- added U7: TLV9062IDR, TLV9062:D0008A_N, F.Cu at (198.4, 76.2)
Routing:
- net Net-(U7A-IN+): track 29.2 -> 116.7 mm
- net /Audio In Sum/AUDIO_IN_R_SUMMED: track 21.2 -> 84.7 mm
- net (no net): track 16.7 -> 61.7 mm
- net /CONN_4_AI_DIO0: track 13.2 -> 52.7 mm
- net /CONN_7_AI_DIO0: track 12.9 -> 51.7 mm
- net /CONN_6_AI_DIO0: track 11.8 -> 47.3 mm
- net /CONN_2_AI_DIO0: track 11.8 -> 47.0 mm
- net /CONN_1_AI_DIO0: track 11.0 -> 44.1 mm
- net /CONN_5_AI_DIO0: track 10.9 -> 43.4 mm
- net /CONN_3_AI_DIO0: track 10.6 -> 42.3 mm
- net Net-(U7B-IN+): track 9.30 -> 37.2 mm
- net Net-(U7B-IN-): track 7.30 -> 29.2 mm
- net Net-(U7B-OUT): track 5.55 -> 22.2 mm
- net Net-(U7A-OUT): track 3.76 -> 15.0 mm
- net /Audio In Sum/AUDIO_IN_L_SUMMED: track 3.57 -> 14.3 mm
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Other:
- board size 56.8 x 65 mm -> 412.5 x 65 mm
- board text added: "0 1"
- board text added: "0 1 2 3"
- board text added: "0 1 2 3 4 5 6 7 8 9"
- board text added: "4 5 6 7"
- board text added: "7 6 5 4 3 2 1 0"
- board text added: "9 8 7 6 5 4 3 2 1 0"
- board text added: "Analog O"
- board text added: "Audio In"
- board text added: "Audio Out"
- board text added: "GND AI 3.3V"
- board text added: "GND AO 3.3V"
- board text added: "GND AudI"
- board text added: "GND AudIAux"
- board text added: "GND AudO"
- board text added: "GND DIO"
- board text added: "GND VIN"
- board text added: "L R"
- board text added: "Left Right"
- board text added: "MIDI IN"
- board text added: "MIDI OUT"
