File: _autosave-DaisySeedBreakout.kicad_pcb (KiCad board)
At the start: 4 copper layers, 39.3 x 60.7 mm, 114 parts, among them J1 Conn_01x03, J10 Conn_01x03, J11 Conn_01x02, J12 Conn_01x02, J13 Conn_01x02, J14 Conn_01x03, J15 USB_B_Micro, J16 Conn_01x02, J17 Conn_01x02, J18 Conn_02x04, J19 Conn_01x06, J2 Conn_01x02, J20 Conn_01x04, J21 Conn_02x04, J23 Pins_02x10_P2.54mm_TH, J24 Conn_01x10, J25 Conn_01x02, J26 Conn_01x02, J3 Conn_01x03, J4 5027740891, J5 Conn_01x04, J6 Conn_01x02, J7 Conn_01x04, J8 Conn_01x02, J9 Conn_01x02, U1 H11L1M, U10 TPD2EUSB30ADRTR, U2 MAX4466EXK_T, U4 LIS2DE12, U7 TLV9062IDR

Commit message: some PCB cleanup
Routing:
- net +3.3V: track 107.1 -> 124.3 mm, vias 14 -> 15
- net Net-(A1-USB_ID): track 9.06 -> 3.75 mm
- net GND: track 85.6 -> 88.0 mm, vias 121 -> 125
- net /SD_CMD: track 10.4 -> 8.49 mm
- net +5V: track 18.5 -> 19.0 mm, vias 7 -> 6
- net /SD_D3: vias 2 -> 1
