File: DaisySeedBreakout.kicad_sch (KiCad schematic)
At the start: 35 parts, among them J10 Conn_01x03, J11 Conn_01x02, J12 Conn_01x02, J13 Conn_01x02, J14 Conn_01x03, J15 USB_B_Micro, J16 Conn_01x03, J18 Conn_02x04, J19 Conn_01x06, J2 Conn_01x02, J20 Conn_01x04, J21 Conn_02x04, J22 Conn_01x02, J5 Conn_01x04, J6 Conn_01x02, J7 Conn_01x04, J8 Conn_01x02, J9 Pins_02x10_P2.54mm_TH, U10 TPD2EUSB30ADRTR

Commit message: Layout routed, no DRC yet
Parts:
- removed J16: Conn_01x03, HeadersWithSolderHoles:PinHeader_1x03_P2.54mm_Vertical_Female_WithSolderHoles, symbol 4ms_Connector:Conn_01x03
- removed J22: Conn_01x02, 1x2FemaleVertical:PinHeader_1x02_P2.54mm_VerticalFemale, symbol 4ms_Connector:Conn_01x02
- removed J9: Pins_02x10_P2.54mm_TH, HeadersWithSolderHoles:PinHeader_3x10_P2.54mm_Vertical, symbol 3x10HeaderWithSolderHoles:Pins_03x10_P2.54mm_TH_SolderHoles
- added C16: 0.1uF, Capacitor_SMD:C_0402_1005Metric, symbol Device:C
- added J16, J25, J26, J9: Conn_01x02, 1x2FemaleVertical:PinHeader_1x02_P2.54mm_VerticalFemale, symbol 4ms_Connector:Conn_01x02
- added J23: Pins_02x10_P2.54mm_TH, 2x10FemaleHeader:PinHeader_2x10_P2.54mm_Vertical, symbol Ultralibrarian_modified_symbols:Pins_02x10_P2.54mm_TH
- added J24: Conn_01x10, Connector_PinHeader_2.54mm:PinHeader_1x10_P2.54mm_Vertical, symbol Connector_Generic:Conn_01x10
- added Z2: RSX501LAM20TR, DIO_RB050LAM_ROM, symbol 2023-10-01_23-34-18:RSX501LAM20TR
- J10, J14: footprint HeadersWithSolderHoles:PinHeader_1x03_P2.54mm_Vertical_Female_WithSolderHoles -> FemaleHeaders:PinHeader_1x03_P2.54mm_Vertical_Female
- J11, J12, J13, J2: footprint HeadersWithSolderHoles:PinHeader_1x02_P2.54mm_VerticalFemale_WithSolderHoles -> 1x2FemaleVertical:PinHeader_1x02_P2.54mm_VerticalFemale
- J18, J21: footprint HeadersWithSolderHoles:PinHeader_2x04_P2.54mm_Vertical_Female -> FemaleHeaders:PinHeader_2x04_P2.54mm_Vertical_Female
Connections:
- net +3.3V: now also C10.1, C2.1, C6.1, C8.1, J10.3 (Pin_3), J14.3 (Pin_3), J23.10, J23.12, J23.14, J23.16, J23.18, J23.2, J23.20, J23.4, J23.6, J23.8, J25.1 (Pin_1), J25.2 (Pin_2), J26.1 (Pin_1), J26.2 (Pin_2)
- net +3.3VA: no longer C10.1, C2.1, C6.1, C8.1, J10.3 (Pin_3), J14.3 (Pin_3)
- net +5V: now also A1.39 (VIN), C15.1, J5.1 (Pin_1), Z1.2, C16.1, J16.1 (Pin_1), J16.2 (Pin_2), J9.1 (Pin_1), J9.2 (Pin_2), Z2.2
- net AI_0: now also J24.10 (Pin_10)
- net AI_1: now also J24.9 (Pin_9)
- net AI_2: now also J24.8 (Pin_8)
- net AI_3: now also J24.7 (Pin_7)
- net AI_4: now also J24.6 (Pin_6)
- net AI_5: now also J24.5 (Pin_5)
- net AI_6: now also J24.4 (Pin_4)
- net AI_7: now also J24.3 (Pin_3)
- net AI_8: now also J24.2 (Pin_2)
- net AI_9: now also J24.1 (Pin_1)
- net GND: now also C16.2, J23.1, J23.11, J23.13, J23.15, J23.17, J23.19, J23.3, J23.5, J23.7, J23.9
- net USB_n: now also U10.2 (D-); no longer U10.1 (D+)
- net USB_p: now also U10.1 (D+); no longer U10.2 (D-)
- net at J15.1 (VBUS): now also Z2.1
Other:
- note added: "3.3V Out"
- note added: "5V In"
- note added: "5V Out"
- note added: "Analog Input"
- note added: "Analog Output"
- note added: "DIO"
- note added: "I2C, UART, SPI Headers"
- moved on the sheet: C10, C2, C6, C8, J10, J14, J15, J18, J19, J20, J21, J5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

Commit message: PCB cleanup, added accelerometer as easy sensor to begin with
Parts:
- added C18: 0.1uF, Capacitor_SMD:C_0402_1005Metric, symbol Device:C
- added C7: 0.1uF, Capacitor_SMD:C_0402_1005Metric, symbol Device:C_Small
- added D1: D_Schottky, Diode_SMD:D_0402_1005Metric, symbol Device:D_Schottky_Small
- added J1, J3: Conn_01x03, FemaleHeaders:PinHeader_1x03_P2.54mm_Vertical_Female, symbol 4ms_Connector:Conn_01x03
- added R34: DNP, Resistor_SMD:R_0402_1005Metric, symbol Device:R_US
- added R52: 10, Resistor_SMD:R_0402_1005Metric, symbol Device:R_US
- added R53: 33, Resistor_SMD:R_0402_1005Metric, symbol Device:R_US
- added R54: 220, Resistor_SMD:R_0402_1005Metric, symbol Device:R_US
- added R55: 270, Resistor_SMD:R_0402_1005Metric, symbol Device:R_US
- added U1: H11L1M, digikey-footprints:DIP-6_W7.62mm, symbol dk_Optoisolators-Logic-Output:H11L1M
- added U4: LIS2DE12, Package_LGA:LGA-12_2x2mm_P0.5mm, symbol Sensor_Motion:LIS2DE12
Connections:
- net +3.3V: now also C18.1, C7.1, R53.1, R55.2, U1.6 (VCC), U4.10 (Vdd_IO), U4.2 (~{CS}), U4.9 (Vdd)
- net DIO4_SCL_RX: now also U4.1 (SCL/SPC)
- net DIO5_SDA_TX: now also U4.4 (SDA/SDI)
- net GND: now also C18.2, C7.2, J1.1 (Pin_1), J3.1 (Pin_1), R34.1, U1.5 (GND), U4.5 (RES), U4.6 (GND), U4.7 (GND), U4.8 (GND)
- net MIDI_UART_RX: now also R55.1, U1.4 (VO)
- net MIDI_UART_TX: now also R52.1
- net HEADER_5V: now reaches J6.2 (Pin_2), Z1.1
- net USB_5V: now reaches J15.1 (VBUS), Z2.1
- net Audio In/AUDIO_IN_L_CONN renamed Audio_IN_L_CONN
- net Audio In/AUDIO_IN_L_SUMMED renamed Audio_IN_1
- net Audio In/AUDIO_IN_R_CONN renamed Audio_IN_R_CONN
- net Audio In/AUDIO_IN_R_SUMMED renamed Audio_IN_2
- net Audio Out/AUDIO_OUT_L renamed Audio_OUT_1
- net Audio Out/AUDIO_OUT_L_EXT renamed Audio_OUT_L_CONN
- net Audio Out/AUDIO_OUT_R renamed Audio_OUT_2
- net Audio Out/AUDIO_OUT_R_EXT renamed Audio_OUT_R_CONN
- net Condensor Microphone/AUDIO_OUT renamed Mic_OUT
- net microSD/CLK renamed SD_CLK
- net microSD/CMD renamed SD_CMD
- net microSD/D0 renamed SD_D0
- net microSD/D1 renamed SD_D1
- net microSD/D2 renamed SD_D2
- net microSD/D3 renamed SD_D3
- new net: R34.2, U4.3 (SA0/SDO)
- new net MIDI_IN_CONN: D1.2 (A), J3.2 (Pin_2), U1.2
- new net MIDI_IN_CONN_R: J3.3 (Pin_3), R54.2
- new net MIDI_IN_Diode: D1.1 (K), R54.1, U1.1
- new net MIDI_TX_CONN: J1.2 (Pin_2), R52.2
- new net MIDI_TX_PWR: J1.3 (Pin_3), R53.2
- no-connect marks 0 -> 2
Other:
- removed sheet MIDI_IN
- removed sheet MIDI_OUT
- note added: "DIO Headers"
- note added: "MIDI IN"
- note added: "MIDI OUT"
- note added: "USB 2.0 Host"
- note removed: "DIO"
- note removed: "ESD Protection?"
- note removed: "USB 2.0"
- moved on the sheet: C16, J15, J16, J18, J19, J2, J20, J21, J25, J26, J5, J6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
