File: _autosave-DaisySeedBreakout.kicad_sch (KiCad schematic)
At the start: 55 parts, among them J1 Conn_01x03, J10 Conn_01x03, J11 Conn_01x02, J12 Conn_01x02, J13 Conn_01x02, J14 Conn_01x03, J15 USB_B_Micro, J16 Conn_01x02, J18 Conn_02x04, J19 Conn_01x06, J2 Conn_01x02, J20 Conn_01x04, J21 Conn_02x04, J23 Pins_02x10_P2.54mm_TH, J24 Conn_01x10, J25 Conn_01x02, J26 Conn_01x02, J3 Conn_01x03, J5 Conn_01x04, J6 Conn_01x02, J7 Conn_01x04, J8 Conn_01x02, J9 Conn_01x02, U1 H11L1M, U10 TPD2EUSB30ADRTR, U4 LIS2DE12

Commit message: making way to generate digikey and mouser boms...work in progress
Parts:
- H1, H2, H3, H4: value MountingHole -> DNP
Changed lines of the file:
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@@
     )
     (property "Value" "GND" (at 250.19 234.95 0)
-      (effects (font (size 1.27 1.27)))
+      (effects (font (size 1.27 1.27)) hide)
     )
     (property "Footprint" "" (at 252.73 235.585 0)
@@
     )
     (property "Value" "GND" (at 260.35 26.67 0)
-      (effects (font (size 1.27 1.27)))
+      (effects (font (size 1.27 1.27)) hide)
     )
     (property "Footprint" "" (at 260.35 21.59 0)
@@
     )
     (property "Value" "GND" (at 236.22 26.67 0)
-      (effects (font (size 1.27 1.27)))
+      (effects (font (size 1.27 1.27)) hide)
     )
     (property "Footprint" "" (at 236.22 21.59 0)
@@
     )
     (property "Value" "GND" (at 347.98 217.805 0)
-      (effects (font (size 1.27 1.27)))
+      (effects (font (size 1.27 1.27)) hide)
     )
     (property "Footprint" "" (at 345.44 218.44 0)
@@
     )
     (property "Value" "GND" (at 234.95 191.77 0)
-      (effects (font (size 1.27 1.27)))
+      (effects (font (size 1.27 1.27)) hide)
     )
     (property "Footprint" "" (at 237.49 192.405 0)
@@
     )
     (property "Value" "GND" (at 88.9 254 0)
-      (effects (font (size 1.27 1.27)))
+      (effects (font (size 1.27 1.27)) hide)
     )
     (property "Footprint" "" (at 92.71 252.73 0)
@@
     )
     (property "Value" "GND" (at 397.002 97.536 0)
-      (effects (font (size 1.27 1.27)))
+      (effects (font (size 1.27 1.27)) hide)
     )
     (property "Footprint" "" (at 394.97 97.79 0)
@@
       (effects (font (size 1.27 1.27)) (justify left))
     )
-    (property "Value" "MountingHole" (at 244.348 22.86 0)
+    (property "Value" "DNP" (at 244.348 22.86 0)
       (effects (font (size 1.27 1.27)) (justify left))
     )
@@
     )
     (property "Value" "GND" (at 128.27 254 0)
-      (effects (font (size 1.27 1.27)))
+      (effects (font (size 1.27 1.27)) hide)
     )
     (property "Footprint" "" (at 132.08 252.73 0)
@@
     )
     (property "Value" "GND" (at 45.72 254 0)
-      (effects (font (size 1.27 1.27)))
+      (effects (font (size 1.27 1.27)) hide)
     )
     (property "Footprint" "" (at 49.53 252.73 0)
@@
       (effects (font (size 1.27 1.27)) (justify left))
     )
-    (property "Value" "MountingHole" (at 268.478 22.86 0)
+    (property "Value" "DNP" (at 268.478 22.86 0)
       (effects (font (size 1.27 1.27)) (justify left))
     )
@@
     )
     (property "Value" "GND" (at 260.35 35.56 0)
-      (effects (font (size 1.27 1.27)))
+      (effects (font (size 1.27 1.27)) hide)
     )
     (property "Footprint" "" (at 260.35 30.48 0)
@@
     )
     (property "Value" "GND" (at 64.77 115.824 0)
-      (effects (font (size 1.27 1.27)))
+      (effects (font (size 1.27 1.27)) hide)
     )
     (property "Footprint" "" (at 66.675 115.57 0)
@@
     )
     (property "Value" "GND" (at 192.405 136.525 0)
-      (effects (font (size 1.27 1.27)))
+      (effects (font (size 1.27 1.27)) hide)
     )
     (property "Footprint" "" (at 190.5 135.89 0)
@@
     )
     (property "Value" "GND" (at 366.649 59.055 0)
-      (effects (font (size 1.27 1.27)))
+      (effects (font (size 1.27 1.27)) hide)
     )
     (property "Footprint" "" (at 367.03 54.61 0)
@@
     )
     (property "Value" "GND" (at 40.64 187.96 0)
-      (effects (font (size 1.27 1.27)))
+      (effects (font (size 1.27 1.27)) hide)
     )
     (property "Footprint" "" (at 40.64 182.88 0)
@@
     )
     (property "Value" "GND" (at 347.98 203.2 0)
-      (effects (font (size 1.27 1.27)))
+      (effects (font (size 1.27 1.27)) hide)
     )
     (property "Footprint" "" (at 345.44 203.835 0)
@@
       (effects (font (size 1.27 1.27)) (justify left))
     )
-    (property "Value" "MountingHole" (at 268.478 31.75 0)
+    (property "Value" "DNP" (at 268.478 31.75 0)
       (effects (font (size 1.27 1.27)) (justify left))
     )
@@
     )
     (property "Value" "GND" (at 234.95 257.81 0)
-      (effects (font (size 1.27 1.27)))
+      (effects (font (size 1.27 1.27)) hide)
     )
     (property "Footprint" "" (at 234.95 252.73 0)
@@
     )
     (property "Value" "GND" (at 52.832 200.66 0)
-      (effects (font (size 1.27 1.27)))
+      (effects (font (size 1.27 1.27)) hide)
     )
     (property "Footprint" "" (at 50.292 200.025 0)
@@
       (effects (font (size 1.27 1.27)) (justify left))
     )
-    (property "Value" "MountingHole" (at 244.348 31.75 0)
+    (property "Value" "DNP" (at 244.348 31.75 0)
       (effects (font (size 1.27 1.27)) (justify left))
     )
@@
     )
     (property "Value" "GND" (at 344.17 101.6 0)
-      (effects (font (size 1.27 1.27)))
+      (effects (font (size 1.27 1.27)) hide)
     )
     (property "Footprint" "" (at 346.71 101.6 0)
@@
     )
     (property "Value" "GND" (at 161.925 255.778 0)
-      (effects (font (size 1.27 1.27)))
+      (effects (font (size 1.27 1.27)) hide)
     )
     (property "Footprint" "" (at 160.02 255.143 0)
@@
     )
     (property "Value" "GND" (at 267.97 235.585 0)
-      (effects (font (size 1.27 1.27)))
+      (effects (font (size 1.27 1.27)) hide)
     )
     (property "Footprint" "" (at 270.51 236.22 0)
@@
     )
     (property "Value" "GND" (at 69.85 90.17 0)
-      (effects (font (size 1.27 1.27)))
+      (effects (font (size 1.27 1.27)) hide)
     )
     (property "Footprint" "" (at 67.31 89.535 0)
@@
     )
     (property "Value" "GND" (at 236.22 35.56 0)
-      (effects (font (size 1.27 1.27)))
+      (effects (font (size 1.27 1.27)) hide)
     )
     (property "Footprint" "" (at 236.22 30.48 0)
@@
     )
     (property "Value" "GND" (at 251.46 254 0)
-      (effects (font (size 1.27 1.27)))
+      (effects (font (size 1.27 1.27)) hide)
     )
     (property "Footprint" "" (at 251.46 248.92 0)
@@
     )
     (property "Value" "GND" (at 363.22 208.28 0)
-      (effects (font (size 1.27 1.27)))
+      (effects (font (size 1.27 1.27)) hide)
     )
     (property "Footprint" "" (at 365.76 208.915 0)
@@
     )
     (property "Value" "GND" (at 208.28 260.35 0)
-      (effects (font (size 1.27 1.27)))
+      (effects (font (size 1.27 1.27)) hide)
     )
     (property "Footprint" "" (at 208.28 255.27 0)
