File: DaisySeedAccessories/DaisySeedAccessories/ArduinoCompanion.kicad_sch (KiCad schematic)
At the start: 0 parts

Commit message: simplified design, rely on external boards more to cover those cases
Parts:
- added C29 (x4): 0.1uF, Capacitor_SMD:C_0402_1005Metric, symbol Device:C
- added R85: 33.2, Resistor_SMD:R_0402_1005Metric, symbol Device:R_US
- added U4: ATMEGA1608-MFR, atmega:VQFN32_RXB_MCH-M, symbol 2023-09-29_01-38-21:ATMEGA1608-MFR
- added U6: DSC6001CE2A-010.0000, DFN4_3.2X2.5_MCH, symbol 2023-09-30_01-44-26:DSC6001CE2A-010.0000
Connections:
- new net: R85.2, U4.30 (PA0(EXTCLK)_TXD)
- new net: R85.1, U6.3 (OUT)
- new net GND: C29.2, C29.2, C29.2, C29.2, U4.19 (GND), U4.29 (GND), U4.33 (GND), U6.2 (GND)
- new net GPIO: U4.31 (PA1_RXD)
- new net GPIO_AIN0: U4.10 (PD0_AIN0)
- new net GPIO_AIN1: U4.11 (PD1_AIN1)
- new net GPIO_AIN14: U4.24 (PF4_AIN14)
- new net GPIO_AIN15: U4.25 (PF5_AIN15)
- new net GPIO_AIN2: U4.12 (PD2_AIN2)
- new net GPIO_AIN3: U4.13 (PD3_AIN3)
- new net GPIO_AIN4: U4.14 (PD4_AIN4)
- new net GPIO_AIN5: U4.15 (PD5_AIN5)
- new net GPIO_AIN6: U4.16 (PD6_AIN6)
- new net GPIO_AIN7: U4.17 (PD7_AIN7)
- new net I2C0_SCL: U4.1 (PA3_SCL)
- new net I2C0_SDA: U4.32 (PA2_SDA)
- new net I2C1_SCL_SPI1_CLK: U4.8 (PC2_SCK_SDA)
- new net I2C1_SCL_SPI1_CS: U4.9 (PC3_SS_SCL)
- new net I2C2_SCL: U4.23 (PF3_SCL)
- new net I2C2_SDA: U4.22 (PF2_SDA)
- new net RESET_n: U4.26 (PF6_RESET)
- new net SPI0_CS: U4.5 (PA7_SS)
- new net SPI0_SCLK: U4.4 (PA6_SCK)
- new net UART0_RXD_SPI0_MISO: U4.3 (PA5_MISO_RXD)
- new net UART0_TXD_SPI0_MOSI: U4.2 (PA4_MOSI_TXD)
- new net UART1_RXD_SPI1_MISO: U4.7 (PC1_RXD)
- new net UART1_TXD_SPI1_MOSI: U4.6 (PC0_TXD)
- new net UART2_RXD: U4.21 (PF1(TOSC2)_RXD)
- new net UART2_TXD: U4.20 (PF0(TOSC1)_TXD)
- new net UDPI: U4.27 (UPDI)
- new net VCC: C29.1, C29.1, C29.1, C29.1, U4.18 (AVDD), U4.28 (VDD), U6.1 (OE), U6.4 (VDD)
