File: DaisySeedAccessories/DaisySeedAccessories/SpeakerDriver20W.kicad_sch (KiCad schematic)
At the start: 0 parts

Commit message: simplified design, rely on external boards more to cover those cases
Parts:
- added C10, C25: 220pF, Capacitor_SMD:C_0402_1005Metric, symbol Device:C
- added C25 (x5): 1u, Capacitor_SMD:C_0603_1608Metric, symbol Device:C
- added C32: 860020474014, CAP_WCAP-ATG5_8x11.5_WRE, symbol 2023-10-01_19-18-23:860020474014
- added C6 (x3): 0.1uF, Capacitor_SMD:C_0603_1608Metric, symbol Device:C
- added FB1, FB3: MPZ1608S221ATA00, digikey-footprints:0603, symbol dk_Ferrite-Beads-and-Chips:MPZ1608S221ATA00
- added R8 (x2): 4.7k, Resistor_SMD:R_0402_1005Metric, symbol Device:R_US
- added R8: 0, Resistor_SMD:R_0402_1005Metric, symbol Device:R_US
- added U2: PAM8320RDR, SO-16EP_3P9X9P9_DIO, symbol 2023-10-01_02-32-05:PAM8320RDR
Connections:
- new net: C25.2, FB1.1, U2.10 (OUTP)
- new net: C25.1, U2.4 (VCM)
- new net: C25.1, U2.7 (VCLAMP)
- new net: C25.2, FB3.1, U2.15 (OUTN)
- new net: C25.1, U2.14 (BSN)
- new net: C25.2, R8.1
- new net: C25.1, U2.11 (BSP)
- new net: R8.2, U2.3 (IN)
- new net GND: C10.2, C25.2, C25.2, C25.2, C32.1, C6.2, C6.2, C6.2, R8.2, R8.2, U2.12 (MUTE), U2.16 (PGNDN), U2.5 (AGND), U2.6 (AGND), U2.9 (PGNDP)
- new net IN: C25.1
- new net OUT_N: C10.1, FB3.2, R8.1
- new net OUT_P: C25.1, FB1.2, R8.1
- new net SHUTDOWN: U2.2 (SDN)
- new net VCC: C32.2, C6.1, C6.1, C6.1, U2.1 (PVCCN), U2.13 (AVCC), U2.8 (PVCCP)
- no-connect marks 0 -> 1
